File: design/temp.kicad_sch (KiCad schematic)
At the start: 3 parts

Commit message: v 4.13 produced by jlcpcb
Some serious issues with usb connectors facing the caps. Working fine
otherwise
Parts:
- C41: JLCPCB (none) -> C23630
- R1: mpn (none) -> NCP18XH103F03RB
Changed lines of the file:
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@@
 (kicad_sch
-	(version 20231120)
+	(version 20250114)
 	(generator "eeschema")
-	(generator_version "8.0")
+	(generator_version "9.0")
 	(paper "A4")
 	(title_block
 		(title "BLDC Driver 4.11")
 		(date "21 aug 2015")
-		(rev "4.12")
+		(rev "${version}")
 		(company "Benjamin Vedder")
 	)
@@
 		(shape input)
 		(at 115.57 95.25 0)
-		(fields_autoplaced yes)
 		(effects
 			(font
@@
 			)
 		)
+		(property "mpn" "NCP18XH103F03RB"
+			(at 111.76 86.36 90)
+			(effects
+				(font
+					(size 1.27 1.27)
+				)
+				(hide yes)
+			)
+		)
 		(pin "1"
 		)
@@
 			(at 105.41 104.14 0)
 			(effects
+				(font
+					(size 1.27 1.27)
+				)
+				(hide yes)
+			)
+		)
+		(property "JLCPCB" "C23630"
+			(at 105.41 104.14 0)
+			(effects
